Commit message: added gazebo plugins and fix all inertial values

File: description/robots/rm3_sherpa_omni.urdf.xacro (robot description, xacro)
@@ -13,20 +13,50 @@
 		      </geometry>
 		</visual>
-		<collision>
-			<origin rpy="0.0 0.0 0.0" xyz="0.0 0.0 ${chassis_field_height}"/>
-			<geometry>
-				<box size="0.001 0.001 0.001"/>
-			</geometry>
-		</collision>
+<!--		<collision>-->
+<!--			<origin rpy="0.0 0.0 0.0" xyz="0.0 0.0 ${chassis_field_height}"/>-->
+<!--			<geometry>-->
+<!--				<box size="0.001 0.001 0.001"/>-->
+<!--			</geometry>-->
+<!--		</collision>-->
 	</link>
-	<joint name="${prefix}base_footprint_joint" type="fixed">
+<!--	<joint name="${prefix}base_footprint_joint" type="fixed">-->
+<!--		<parent link="baselink"/>-->
+<!--		<child link="${prefix}base_link"/>-->
+<!--<!- -        <origin xyz="0.0 0.0 0.0"/>- ->-->
+<!--		<origin xyz="0.622 0.0 0.0"/>-->
+<!--	</joint>-->
+<!--	-->
+<!--<!- - Chassis - ->-->
+<!--	<link name="${prefix}base_link">-->
+<!--		<visual>-->
+<!--			<origin rpy="0.0 0.0 ${PI}" xyz="0.0 0.0 ${chassis_z/2-0.0150}"/>-->
+<!--			<geometry>-->
+<!--<mesh filename="package://rm3_sherpa_description/description/meshes/rbsherpa_hl_base_tank.dae" />-->
+<!--			</geometry>-->
+<!--		</visual>-->
+<!--     -->
+<!--		<collision>-->
+<!--			<origin rpy="0.0 0.0 0.0" xyz="0.0 0.0 ${chassis_field_height+chassis_z/2}"/>-->
+<!--			<geometry>-->
+<!--				<box size="${chassis_x} ${chassis_y} ${chassis_z}"/>-->
+<!--			</geometry>-->
+<!--		</collision>-->
+<!--     -->
+<!--		<inertial> -->
+<!--			<origin rpy="0.0 0.0 0.0" xyz="0.0 0.0 ${chassis_field_height+chassis_z/2}"/>-->
+<!--			<mass value="${mass}"/>-->
+<!--			<box_inertia  m="${mass}" h="${chassis_x}" w ="${chassis_y}" d="${chassis_z}"/>-->
+<!--		</inertial>-->
+<!--	</link>-->
+<!--	-->
+<!--	<gazebo reference="${prefix}base_link"><material>Gazebo/Red</material></gazebo>-->
+    <joint name="${prefix}base_footprint_joint" type="fixed">
 		<parent link="baselink"/>
 		<child link="${prefix}base_link"/>
-<!--        <origin xyz="0.0 0.0 0.0"/>-->
 		<origin xyz="0.622 0.0 0.0"/>
 	</joint>
 <!-- Chassis -->
 	<link name="${prefix}base_link">
-		<visual>
+        <visual>-->
 			<origin rpy="0.0 0.0 ${PI}" xyz="0.0 0.0 ${chassis_z/2-0.0150}"/>
 			<geometry>
@@ -34,4 +64,10 @@
 			</geometry>
 		</visual>
+<!--		<visual>-->
+<!--			<origin rpy="0.0 0.0 0.0" xyz="0.0 0.0 ${chassis_field_height+chassis_z/2}"/>-->
+<!--			<geometry>-->
+<!--				<box size="${chassis_x} ${chassis_y} ${chassis_z}"/>-->
+<!--			</geometry>-->
+<!--		</visual>-->
 		<collision>
 			<origin rpy="0.0 0.0 0.0" xyz="0.0 0.0 ${chassis_field_height+chassis_z/2}"/>
@@ -42,9 +78,12 @@
 		<inertial>
 			<origin rpy="0.0 0.0 0.0" xyz="0.0 0.0 ${chassis_field_height+chassis_z/2}"/>
-			<mass value="${mass}"/>
-			<box_inertia  m="${mass}" h="${chassis_x}" w ="${chassis_y}" d="${chassis_z}"/>
+			<mass value="1"/>
+			<box_inertia  m="1" h="${chassis_x}" w ="${chassis_y}" d="${chassis_z}"/>
 		</inertial>
 	</link>
-	<gazebo reference="${prefix}base_link"><material>Gazebo/Red</material></gazebo>
+  <gazebo reference="${prefix}base_link">
+    <material>Gazebo/Red</material>
+    <mu1 value="${mu_1}"/>
+  </gazebo>
 <!-- ros_control plugin -->
 	<gazebo>
@@ -62,3 +101,21 @@
 <xacro:include filename="$(find rm3_sherpa_description)/description/urdf/sherpa_wheel.xacro"/>
 <xacro:include filename="$(find rm3_sherpa_description)/description/urdf/sensors.xacro"/>
+  <!-- GAZEBO -->
+  <!-- ros_control plugin -->
+  <gazebo>
+    <plugin name="ground_truth" filename="libgazebo_ros_p3d.so">
+      <alwaysOn>true</alwaysOn>
+      <updateRate>100.0</updateRate>
+      <bodyName>baselink</bodyName>
+      <topicName>/odom_gps</topicName>
+      <gaussianNoise>0.00</gaussianNoise>
+      <frameName>/map</frameName>
+      <xyzOffsets>0 0 0</xyzOffsets>
+      <rpyOffsets>0 0 0</rpyOffsets>
+    </plugin>
+    <!-- ros_control plugin -->
+    <plugin name="gazebo_ros_control" filename="libgazebo_ros_control.so">
+          <legacyModeNS>true</legacyModeNS>
+          </plugin>
+  </gazebo>
 </robot>

File: description/urdf/arm.xacro (robot description, xacro)
@@ -20,9 +20,9 @@
     <inertial>
       <origin rpy="0.0 0.0 0.0" xyz="0.0 0.0 ${(1.888-(chassis_z+chassis_field_height))/2}" />
-      <mass value="1.0" />
-      <box_inertia  m="1.0" h="${lsp_x}" w ="${lsp_y}" d="${(1.888-(chassis_z+chassis_field_height))}"/>
+      <mass value="0.5" />
+      <box_inertia  m="0.5" h="${lsp_x}" w ="${lsp_y}" d="${(1.888-(chassis_z+chassis_field_height))}"/>
     </inertial>
 </link>
-<gazebo reference="${prefix}torso_elevator_link"><material>Gazebo/Black</material></gazebo>
+<gazebo reference="${prefix}torso_elevator_link"><material>Gazebo/DarkGrey</material></gazebo>
 <joint name="fake_torso_elevator_joint" type="fixed">
     <parent link="${prefix}base_link"/>
@@ -39,9 +39,9 @@
     <inertial>
       <origin rpy="0.0 0.0 0.0" xyz="0.0 0.0 ${(1.89120-(chassis_z+chassis_field_height))/2}" />
-      <mass value="1.0" />
-      <box_inertia  m="1.0" h="${lsp_x}" w ="${lsp_y}" d="${(1.888-(chassis_z+chassis_field_height))}"/>
+      <mass value="0.5" />
+      <box_inertia  m="0.5" h="${lsp_x}" w ="${lsp_y}" d="${(1.888-(chassis_z+chassis_field_height))}"/>
     </inertial>
 </link>
-<gazebo reference="fake_torso_elevator_link"><material>Gazebo/Black</material></gazebo>
+<gazebo reference="fake_torso_elevator_link"><material>Gazebo/DarkGrey</material></gazebo>
 <!-- Pan -->
 <joint name="${prefix}torso_pantilt_pan_joint" type="revolute">
@@ -61,8 +61,8 @@
     <inertial>
       <origin rpy="0.0 0.0 0.0" xyz="0 0 ${pan_z/2}"/>
-      <mass value="1" />
-      <box_inertia  m="1" h="${pan_x}" w ="${pan_y}" d="${pan_z}"/>
+      <mass value="0.5" />
+      <box_inertia  m="0.5" h="${pan_x}" w ="${pan_y}" d="${pan_z}"/>
     </inertial>
 </link>
-<gazebo reference="${prefix}torso_pantilt_pan_link"><material>Gazebo/Grey</material></gazebo>
+<gazebo reference="${prefix}torso_pantilt_pan_link"><material>Gazebo/DarkGrey</material></gazebo>
 </robot>

File: description/urdf/macros.xacro (robot description, xacro)
@@ -2,72 +2,109 @@
 <!-- Sherpa -->
 <robot name ="sherpa" xmlns:xacro="http://www.ros.org/wiki/xacro">
-<!--from sherpa_ex-->
-<!-- Box Inertia -->
-<xacro:macro name="box_inertia" params="m h w d">
-	<inertia 	ixx="${m*(w*w+d*d)/12}" ixy = "0.0" ixz = "0.0"
-			iyy="${m*(d*d+h*h)/12}" iyz = "0.0"
-			izz="${m*(w*w+h*h)/12}"/>
-</xacro:macro>
-<!-- Cylinder Inertia -->
-<xacro:macro name="cylinder_inertia" params="m r h">
-	<inertia  	ixx="${m*(3*r*r+h*h)/12}" ixy = "0.0" ixz = "0.0"
-			iyy="${m*r*r/2}" iyz = "0.0"
-			izz="${m*(3*r*r+h*h)/12}"/>
-</xacro:macro> <!--modified 10/05/2019 (swapped y and z inertia) -->
-<!-- Parameters -->
-<xacro:property name="PI" value="3.1415926535897931"/>
-<xacro:property name="offset" value="0.0010"/>
-<!-- Chassis Property -->
-<xacro:property name="chassis_x" value="1.64340"/>
-<xacro:property name="chassis_y" value="1.0040"/>
-<xacro:property name="chassis_z" value="0.39440"/>
-<xacro:property name="chassis_field_height" value="0.46990"/>
-<xacro:property name="mass" value="450.0"/>
-<!--added offset of wheels from robotnik model  -->
-<xacro:property name="wheel_steer_offset_x" value="0.622" />
-<xacro:property name="wheel_steer_offset_y" value="0.367" />
-<xacro:property name="wheel_steer_offset_z" value="0.285" />
-<xacro:property name="wheel_traction_offset_x" value="0.0" />
-<xacro:property name="wheel_traction_offset_y" value="0.03" />
-<xacro:property name="wheel_traction_offset_z" value="-0.285" />
-<xacro:property name="track_width" value="0.755620"/>
-<xacro:property name="wheelbase" value="1.24570"/>
-  <!-- Cable Box Property -->
-  <xacro:property name="cb_x" value="0.060"/>
-  <xacro:property name="cb_y" value="0.1750"/>
-  <xacro:property name="cb_z" value="0.550"/>
-  <xacro:property name="cb_origin_x" value="-0.5675"/> <!-- Origin wrt to chassis' frame -->
-  <xacro:property name="cb_origin_y" value="0"/>
-  <xacro:property name="cb_origin_z" value="0.833"/> <!-- Height of the top of the chassis wrt ground -->
-  <!-- Wheel Parameters -->
-  <xacro:property name="steer_z" value="0.060"/>
-  <xacro:property name="steer_radius" value="0.11530"/>
-  <xacro:property name="suspension_x" value="0.080"/>
-  <xacro:property name="suspension_y" value="0.080"/>
-  <xacro:property name="suspension_z" value="0.22560"/>
-  <xacro:property name="wheel_radius" value="0.17430"/>
-  <xacro:property name="wheel_width" value="0.11420"/>
-  <xacro:property name="wheel_mass" value="10.0"/>
-<!-- Sensors -->
-<xacro:property name="sick_front_x" value="1.64340"/>
-<xacro:property name="sick_front_y" value="1.0040"/>
-<xacro:property name="sick_front_z" value="0.2548"/>
-<xacro:property name="sick_rear_x" value="1.64340"/>
-<xacro:property name="sick_rear_y" value="1.0040"/>
-<xacro:property name="sick_rear_z" value="0.2402"/>
-<!-- Arm Parameters -->
-<!-- lift_gun properties --> <!-- represents the total block lift -->
-<xacro:property name="lg_x" value="0.168109"/>
-<xacro:property name="lg_y" value="0.13725"/>
-<xacro:property name="lg_z" value="0.9420"/>
-<xacro:property name="lg_origin_x" value="${cb_origin_x+cb_x/2+lg_x/2}"/> <!-- Origin wrt chassis' frame -->
-<!--<xacro:property name="lg_origin_y" value="0.0"/>-->
-<!--<xacro:property name="lg_origin_z" value="${cb_origin_z}"/> <!- - Height of the top of the chassis wrt ground - ->-->
-<!-- lift_second_part properties -->
-<xacro:property name="lsp_x" value="0.04507"/>
-<xacro:property name="lsp_y" value="0.13725"/>
-<!-- pan properties -->
-<xacro:property name="pan_x" value="0.980915"/>
-<xacro:property name="pan_y" value="0.07"/>
-<xacro:property name="pan_z" value="0.04291"/>
+    <!--from sherpa_ex-->
+    <!-- Box Inertia -->
+    <xacro:macro name="box_inertia" params="m h w d">
+        <inertia 	ixx="${m*(w*w+d*d)/12}" ixy = "0.0" ixz = "0.0"
+        iyy="${m*(d*d+h*h)/12}" iyz = "0.0"
+        izz="${m*(w*w+h*h)/12}"/>
+    </xacro:macro>
+    <!-- Cylinder Inertia USELESS-->
+    <xacro:macro name="cylinder_inertia" params="m r h">
+        <inertia  	ixx="${m*(3*r*r+h*h)/12}" ixy = "0.0" ixz = "0.0"
+        iyy="${m*r*r/2}" iyz = "0.0"
+        izz="${m*(3*r*r+h*h)/12}"/>
+    </xacro:macro> <!--modified 10/05/2019 (swapped y and z inertia) -->
+    <xacro:macro name="default_inertial_wheel" params="mass">
+        <inertial>
+          <origin xyz="0 0 0" rpy="0 0 0"/>
+          <mass value="${mass}"/>
+          <inertia
+	      ixx="0.1" ixy="0.0" ixz="0.0"
+	      iyy="0.1" iyz="0.0"
+	      izz="0.1"/>
+        </inertial>
+    </xacro:macro>
+    <xacro:macro name="default_inertial" params="mass">
+        <inertial>
+          <origin xyz="0 0 0" rpy="0 0 0"/>
+          <mass value="${mass}"/>
+          <inertia
+	      ixx="0.1" ixy="0.0" ixz="0.0"
+	      iyy="0.1" iyz="0.0"
+	      izz="0.1"/>
+        </inertial>
+    </xacro:macro>
+    <xacro:macro name="fake_inertial">
+        <inertial>
+          <origin xyz="0 0 0" rpy="0 0 0"/>
+          <mass value="1e-5"/>
+          <inertia
+	      ixx="1e-6" ixy="0.0" ixz="0.0"
+	      iyy="1e-6" iyz="0.0"
+	      izz="1e-6"/>
+        </inertial>
+    </xacro:macro>
+    <!-- Parameters -->
+    <xacro:property name="PI" value="3.1415926535897931"/>
+    <xacro:property name="offset" value="0.0010"/>
+    <!-- Chassis Property -->
+    <xacro:property name="chassis_x" value="1.64340"/>
+    <xacro:property name="chassis_y" value="1.0040"/>
+    <xacro:property name="chassis_z" value="0.39440"/>
+    <xacro:property name="chassis_field_height" value="0.46990"/>
+    <!--tested-->
+    <!--    <xacro:property name="mass" value="450.0"/>-->
+    <!--new-->
+    <xacro:property name="mass" value="5.0"/>
+    <!--added offset of wheels from robotnik model  -->
+    <xacro:property name="wheel_steer_offset_x" value="0.622" />
+    <xacro:property name="wheel_steer_offset_y" value="0.367" />
+    <xacro:property name="wheel_steer_offset_z" value="0.285" />
+    <xacro:property name="wheel_traction_offset_x" value="0.0" />
+    <xacro:property name="wheel_traction_offset_y" value="0.03" />
+    <xacro:property name="wheel_traction_offset_z" value="-0.285" />
+    <xacro:property name="track_width" value="0.755620"/>
+    <xacro:property name="wheelbase" value="1.24570"/>
+    <!-- Cable Box Property -->
+    <xacro:property name="cb_x" value="0.060"/>
+    <xacro:property name="cb_y" value="0.1750"/>
+    <xacro:property name="cb_z" value="0.550"/>
+    <xacro:property name="cb_origin_x" value="-0.5675"/> <!-- Origin wrt to chassis' frame -->
+    <xacro:property name="cb_origin_y" value="0"/>
+    <xacro:property name="cb_origin_z" value="0.833"/> <!-- Height of the top of the chassis wrt ground -->
+    <!-- Wheel Parameters -->
+    <xacro:property name="steer_z" value="0.060"/>
+    <xacro:property name="steer_radius" value="0.11530"/>
+    <xacro:property name="suspension_x" value="0.080"/>
+    <xacro:property name="suspension_y" value="0.080"/>
+    <xacro:property name="suspension_z" value="0.22560"/>
+    <xacro:property name="wheel_radius" value="0.17430"/>
+    <xacro:property name="wheel_width" value="0.11420"/>
+    <!--tested-->
+    <!--    <xacro:property name="wheel_mass" value="10.0"/>-->
+    <!--new-->
+    <xacro:property name="wheel_mass" value="1.0"/>
+    <!-- Sensors -->
+    <xacro:property name="sick_front_x" value="1.64340"/>
+    <xacro:property name="sick_front_y" value="1.0040"/>
+    <xacro:property name="sick_front_z" value="0.2548"/>
+    <xacro:property name="sick_rear_x" value="1.64340"/>
+    <xacro:property name="sick_rear_y" value="1.0040"/>
+    <xacro:property name="sick_rear_z" value="0.2402"/>
+    <!-- Arm Parameters -->
+    <!-- lift_gun properties --> <!-- represents the total block lift -->
+    <xacro:property name="lg_x" value="0.168109"/>
+    <xacro:property name="lg_y" value="0.13725"/>
+    <xacro:property name="lg_z" value="0.9420"/>
+    <xacro:property name="lg_origin_x" value="${cb_origin_x+cb_x/2+lg_x/2}"/> <!-- Origin wrt chassis' frame -->
+    <!--<xacro:property name="lg_origin_y" value="0.0"/>-->
+    <!--<xacro:property name="lg_origin_z" value="${cb_origin_z}"/> <!- - Height of the top of the chassis wrt ground - ->-->
+    <!-- lift_second_part properties -->
+    <xacro:property name="lsp_x" value="0.04507"/>
+    <xacro:property name="lsp_y" value="0.13725"/>
+    <!-- pan properties -->
+    <xacro:property name="pan_x" value="0.980915"/>
+    <xacro:property name="pan_y" value="0.07"/>
+    <xacro:property name="pan_z" value="0.04291"/>
+    <xacro:property name="mu_1" value="9999999999999999999999999999999" />
 </robot>

File: description/urdf/sensors.xacro (robot description, xacro)
@@ -8,5 +8,6 @@
 			<origin xyz="0 0 0" rpy="0 0 0"/>
 			<geometry>
-				<box size="0.1 0.1 0.1"/>
+<!--				<box size="0.1 0.1 0.1"/>-->
+                <cylinder radius="0.05" length="0.1"/>
 			</geometry>
 		</visual>
@@ -27,5 +28,5 @@
 		<sensor type="ray" name="Sick S300_1">
 			<pose>0 0 0 0 0 0</pose>
-			<visualize>true</visualize>
+			<visualize>false</visualize>
 			<update_rate>12.5</update_rate>
 			<ray>
@@ -49,4 +50,5 @@
 			</plugin>
 		</sensor>
+        <material>Gazebo/Yellow</material>
 	</gazebo>
 <!-- Rear Sick -->
@@ -55,5 +57,6 @@
 			<origin xyz="0 0 0" rpy="0 0 0"/>
 			<geometry>
-				<box size="0.1 0.1 0.1"/>
+<!--				<box size="0.1 0.1 0.1"/>-->
+                <cylinder radius="0.05" length="0.1"/>
 			</geometry>
 		</visual>
@@ -74,5 +77,5 @@
 		<sensor type="ray" name="Sick S300_rear">
 			<pose>0 0 0 0 0 0</pose>
-			<visualize>true</visualize>
+			<visualize>false</visualize>
 			<update_rate>12.5</update_rate>
 			<ray>
@@ -96,4 +99,5 @@
 			</plugin>
 		</sensor>
+	    <material>Gazebo/Yellow</material>
 	</gazebo>
 <!-- GPS -->
@@ -116,5 +120,7 @@
 		</inertial>
 	</link>
-	<gazebo reference="gps_support"><material>Gazebo/Black</material></gazebo>
+	<gazebo reference="gps_support">
+        <material>Gazebo/Black</material>
+    </gazebo>
 	<joint name="gps_joint" type="fixed">
 		<parent link="${prefix}base_link"/>
@@ -172,9 +178,11 @@
 		<inertial>
 			<origin xyz="0 0 0" rpy="0 0 0"/>
-			<mass value="10.0" />
-			<box_inertia  m="10.0" h="0.10" w ="0.20" d="0.150"/>
-		</inertial>
-	</link>
-	<gazebo reference="faro"><material>Gazebo/Grey</material></gazebo>
+			<mass value="1.0" />
+			<box_inertia  m="1.0" h="0.10" w ="0.20" d="0.150"/>
+		</inertial>
+	</link>
+	<gazebo reference="faro">
+        <material>Gazebo/DarkGrey</material>
+    </gazebo>
 <!-- Gimball -->
 	<joint name="arm_yaw_joint" type="fixed">
@@ -191,10 +199,12 @@
 		</visual>
 		<inertial>
-			<mass value="1.0" />
-			<origin xyz="0 0 0" rpy="0 0 0"/>
-			<box_inertia  m="1.0" h="0.040" w ="0.040" d="0.15180"/>
-		</inertial>
-	</link>
-	<gazebo reference="support_yaw"><material>Gazebo/Grey</material></gazebo>
+			<mass value="0.5" />
+			<origin xyz="0 0 0" rpy="0 0 0"/>
+			<box_inertia  m="0.5" h="0.040" w ="0.040" d="0.15180"/>
+		</inertial>
+	</link>
+	<gazebo reference="support_yaw">
+        <material>Gazebo/DarkGrey</material>
+    </gazebo>
 	<joint name="${prefix}gimbal_yaw_joint" type="revolute">
 		<parent link="${prefix}torso_pantilt_pan_link"/>
@@ -212,10 +222,12 @@
 		</visual>
 		<inertial>
-			<mass value="1.0" />
-			<origin xyz="0 0 0" rpy="0 0 0"/>
-			<box_inertia  m="1.0" h="0.340" w ="0.050" d="0.020"/>
-		</inertial>
-	</link>
-	<gazebo reference="${prefix}gimbal_yaw_link"><material>Gazebo/Grey</material></gazebo>
+			<mass value="0.5" />
+			<origin xyz="0 0 0" rpy="0 0 0"/>
+			<box_inertia  m="0.5" h="0.340" w ="0.050" d="0.020"/>
+		</inertial>
+	</link>
+	<gazebo reference="${prefix}gimbal_yaw_link">
+        <material>Gazebo/DarkGrey</material>
+    </gazebo>
 <!--	<joint name="yaw_roll_joint" type="fixed">-->
 <!--		<parent link="yaw"/>-->
@@ -256,10 +268,12 @@
 		</visual>
 		<inertial>
-			<mass value="2.0" />
+			<mass value="0.5" />
 			<origin xyz="0.0 0.0 0.0" rpy="0.0 0.0 0.0"/>
-			<box_inertia  m="2.0" h="0.20" w ="0.340" d="0.050"/>
-		</inertial>
-	</link>
-	<gazebo reference="${prefix}gimbal_roll_link"><material>Gazebo/Grey</material></gazebo>
+			<box_inertia  m="0.5" h="0.20" w ="0.340" d="0.050"/>
+		</inertial>
+	</link>
+	<gazebo reference="${prefix}gimbal_roll_link">
+        <material>Gazebo/DarkGrey</material>
+    </gazebo>
 <!--	<joint name="pitch_support_joint" type="fixed">-->
 <!--		<parent link="roll"/>-->
@@ -322,10 +336,12 @@
 		</visual>
 		<inertial>
-			<mass value="1.0"/>
+			<mass value="0.5"/>
 			<origin xyz="0.0 0.140 0.0" rpy="0.0 0.0 0.0"/>
-			<box_inertia  m="1.0" h="0.0050" w ="0.20" d="0.190"/>
-		</inertial>
-	</link>
-	<gazebo reference="${prefix}gimbal_pitch_link"><material>Gazebo/Grey</material></gazebo>
+			<box_inertia  m="0.5" h="0.0050" w ="0.20" d="0.190"/>
+		</inertial>
+	</link>
+	<gazebo reference="${prefix}gimbal_pitch_link">
+        <material>Gazebo/DarkGrey</material>
+    </gazebo>
 	<joint name="camera_joint" type="fixed">
 		<parent link="${prefix}gimbal_pitch_link"/>
@@ -341,7 +357,7 @@
 		</visual>
 		<inertial>
-			<mass value="1.0" />
+			<mass value="0.5" />
 			<origin xyz="0.0 0.0 0.0" rpy="0.0 0.0 0.0"/>
-			<box_inertia  m="1.0" h="0.020" w ="0.020" d="0.020"/>
+			<box_inertia  m="0.5" h="0.020" w ="0.020" d="0.020"/>
 		</inertial>
 	</link>
@@ -351,4 +367,44 @@
 		<origin xyz="0.11540 0.14610 0.06410" rpy="0.0 0.0 0.0"/>
 	</joint>
+    <!-- camera -->
+    <gazebo reference="camera">
+        <sensor type="camera" name="camera">
+          <update_rate>30.0</update_rate>
+          <camera name="head">
+            <horizontal_fov>1.3962634</horizontal_fov>
+            <image>
+              <width>800</width>
+              <height>800</height>
+              <format>R8G8B8</format>
+            </image>
+            <clip>
+              <near>0.02</near>
+              <far>300</far>
+            </clip>
+            <noise>
+              <type>gaussian</type>
+              <!-- Noise is sampled independently per pixel on each frame.
+                   That pixel's noise value is added to each of its color
+                   channels, which at that point lie in the range [0,1]. -->
+              <mean>0.0</mean>
+              <stddev>0.007</stddev>
+            </noise>
+          </camera>
+          <plugin name="camera_controller" filename="libgazebo_ros_camera.so">
+            <alwaysOn>true</alwaysOn>
+            <updateRate>0.0</updateRate>
+            <cameraName>camera</cameraName>
+            <imageTopicName>image_raw</imageTopicName>
+            <cameraInfoTopicName>camera_info</cameraInfoTopicName>
+            <frameName>camera</frameName>
+            <hackBaseline>0.07</hackBaseline>
+            <distortionK1>0.0</distortionK1>
+            <distortionK2>0.0</distortionK2>
+            <distortionK3>0.0</distortionK3>
+            <distortionT1>0.0</distortionT1>
+            <distortionT2>0.0</distortionT2>
+          </plugin>
+        </sensor>
+      </gazebo>
 	<link name="micasense">
 		<visual>
@@ -359,10 +415,10 @@
 		</visual>
 		<inertial>
-			<mass value="1.0" />
+			<mass value="0.5" />
 			<origin xyz="0.0 0.0 0.0" rpy="0.0 0.0 0.0"/>
-			<box_inertia  m="1.0" h="0.020" w ="0.020" d="0.020"/>
-		</inertial>
-	</link>
-<!-- IMU -->
+			<box_inertia  m="0.5" h="0.020" w ="0.020" d="0.020"/>
+		</inertial>
+	</link>
+    <!-- IMU -->
 	<joint name="imu_joint" type="fixed">
 		<parent link="${prefix}base_link"/>
@@ -402,4 +458,7 @@
 		</inertial>
 	</link>
+    <gazebo reference="${prefix}velodyne_base_link">
+        <material>Gazebo/DarkGrey</material>
+    </gazebo>
 <!--
 	<link name="velodyne_cover">
