Commit message: added URDF model

File: description/robots/rm3_sherpa_omni.urdf (robot description, URDF)
Before this commit: robot sherpa, 24 links, 23 joints
Links:
- added link gps, mass 0.50; visual cylinder length=0.040 radius=0.090
- added link gps_support, mass 0.50; visual cylinder length=0.30 radius=0.0090
- link rbsherpa_hl_base_link: geometry collision box size=1.6434 1.004 0.3944; visual mesh filename=package://rm3_sherpa_description/description/meshes/rbsherp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
Joints:
- added joint gps_joint: type fixed, parent rbsherpa_hl_base_link, child gps, origin xyz=-0.622 0.0 2.050 rpy=0 0 0
- added joint gps_support_joint: type fixed, parent gps, child gps_support, origin xyz=0.0 0.0 -0.15 rpy=0 0 0
- joint rbsherpa_hl_torso_elevator_joint: limit lower=0.0 upper=5 effort=1000 velocity=0.5 -> lower=0.0 upper=2.5 effort=1000 velocity=0.5
