Commit message: added meshes missing

File: description/urdf/sherpa_wheel.xacro (robot description, xacro)
@@ -32,5 +32,5 @@
       <origin rpy="0.0 0.0 0.0" xyz="0.0 0.0 -${steer_z/2-0.0120}"/>
       <geometry>
-        <mesh filename="package://rbsherpa_hl_description/meshes/wheels/rbsherpa_hl_steer_wheel.dae" />
+        <mesh filename="package://rm3_sherpa_description/meshes/rbsherpa_hl_steer_wheel.dae" />
       </geometry>
     </visual>
@@ -62,5 +62,5 @@
       <origin rpy="0.0 ${PI/2} 0.0" xyz="0.0 ${wheel_width/2} 0.0"/>
       <geometry>
-        <mesh filename="package://rbsherpa_hl_description/meshes/wheels/rbsherpa_hl_traction_wheel.dae" />
+        <mesh filename="package://rm3_sherpa_description/meshes/rbsherpa_hl_traction_wheel.dae" />
       </geometry>
 <!--      <origin rpy="0.0 ${PI/2} ${PI/2}" xyz="0.0 ${wheel_width/2} 0.0"/>-->
@@ -125,5 +125,5 @@
       <origin rpy="0.0 0.0 ${PI}" xyz="0.0 0.0 -${steer_z/2-0.0120}"/>
       <geometry>
-        <mesh filename="package://rbsherpa_hl_description/meshes/wheels/rbsherpa_hl_steer_wheel.dae" />
+        <mesh filename="package://rm3_sherpa_description/meshes/rbsherpa_hl_steer_wheel.dae" />
       </geometry>
     </visual>
@@ -154,5 +154,5 @@
       <origin rpy="0.0 ${PI/2} 0.0" xyz="0.0 -${wheel_width/2} 0.0"/>
       <geometry>
-        <mesh filename="package://rbsherpa_hl_description/meshes/wheels/rbsherpa_hl_traction_wheel.dae" />
+        <mesh filename="package://rm3_sherpa_description/meshes/rbsherpa_hl_traction_wheel.dae" />
       </geometry>
     </visual>
@@ -202,5 +202,5 @@
       <origin rpy="0.0 0.0 0.0" xyz="0.0 0.0 -${steer_z/2-0.0120}"/>
       <geometry>
-        <mesh filename="package://rbsherpa_hl_description/meshes/wheels/rbsherpa_hl_steer_wheel.dae" />
+        <mesh filename="package://rm3_sherpa_description/meshes/rbsherpa_hl_steer_wheel.dae" />
       </geometry>
     </visual>
@@ -231,5 +231,5 @@
       <origin rpy="0.0 ${PI/2} 0.0" xyz="0.0 ${wheel_width/2} 0.0"/>
       <geometry>
-        <mesh filename="package://rbsherpa_hl_description/meshes/wheels/rbsherpa_hl_traction_wheel.dae" />
+        <mesh filename="package://rm3_sherpa_description/meshes/rbsherpa_hl_traction_wheel.dae" />
       </geometry>
     </visual>
@@ -279,5 +279,5 @@
       <origin rpy="0.0 0.0 ${PI}" xyz="0.0 0.0 -${steer_z/2-0.0120}"/>
       <geometry>
-        <mesh filename="package://rbsherpa_hl_description/meshes/wheels/rbsherpa_hl_steer_wheel.dae" />
+        <mesh filename="package://rm3_sherpa_description/meshes/rbsherpa_hl_steer_wheel.dae" />
       </geometry>
     </visual>
@@ -308,5 +308,5 @@
       <origin rpy="0.0 ${PI/2} 0.0" xyz="0.0 -${wheel_width/2} 0.0"/>
       <geometry>
-        <mesh filename="package://rbsherpa_hl_description/meshes/wheels/rbsherpa_hl_traction_wheel.dae" />
+        <mesh filename="package://rm3_sherpa_description/meshes/rbsherpa_hl_traction_wheel.dae" />
       </geometry>
     </visual>

Commit message: added meshes missing

File: description/urdf/sherpa_wheel.xacro (robot description, xacro)
@@ -32,5 +32,5 @@
       <origin rpy="0.0 0.0 0.0" xyz="0.0 0.0 -${steer_z/2-0.0120}"/>
       <geometry>
-        <mesh filename="package://rm3_sherpa_description/meshes/rbsherpa_hl_steer_wheel.dae" />
+        <mesh filename="package://rm3_sherpa_description/description/meshes/rbsherpa_hl_steer_wheel.dae" />
       </geometry>
     </visual>
@@ -62,5 +62,5 @@
       <origin rpy="0.0 ${PI/2} 0.0" xyz="0.0 ${wheel_width/2} 0.0"/>
       <geometry>
-        <mesh filename="package://rm3_sherpa_description/meshes/rbsherpa_hl_traction_wheel.dae" />
+        <mesh filename="package://rm3_sherpa_description/description/meshes/rbsherpa_hl_traction_wheel.dae" />
       </geometry>
 <!--      <origin rpy="0.0 ${PI/2} ${PI/2}" xyz="0.0 ${wheel_width/2} 0.0"/>-->
@@ -125,5 +125,5 @@
       <origin rpy="0.0 0.0 ${PI}" xyz="0.0 0.0 -${steer_z/2-0.0120}"/>
       <geometry>
-        <mesh filename="package://rm3_sherpa_description/meshes/rbsherpa_hl_steer_wheel.dae" />
+        <mesh filename="package://rm3_sherpa_description/description/meshes/rbsherpa_hl_steer_wheel.dae" />
       </geometry>
     </visual>
@@ -154,5 +154,5 @@
       <origin rpy="0.0 ${PI/2} 0.0" xyz="0.0 -${wheel_width/2} 0.0"/>
       <geometry>
-        <mesh filename="package://rm3_sherpa_description/meshes/rbsherpa_hl_traction_wheel.dae" />
+        <mesh filename="package://rm3_sherpa_description/description/meshes/rbsherpa_hl_traction_wheel.dae" />
       </geometry>
     </visual>
@@ -202,5 +202,5 @@
       <origin rpy="0.0 0.0 0.0" xyz="0.0 0.0 -${steer_z/2-0.0120}"/>
       <geometry>
-        <mesh filename="package://rm3_sherpa_description/meshes/rbsherpa_hl_steer_wheel.dae" />
+        <mesh filename="package://rm3_sherpa_description/description/meshes/rbsherpa_hl_steer_wheel.dae" />
       </geometry>
     </visual>
@@ -231,5 +231,5 @@
       <origin rpy="0.0 ${PI/2} 0.0" xyz="0.0 ${wheel_width/2} 0.0"/>
       <geometry>
-        <mesh filename="package://rm3_sherpa_description/meshes/rbsherpa_hl_traction_wheel.dae" />
+        <mesh filename="package://rm3_sherpa_description/description/meshes/rbsherpa_hl_traction_wheel.dae" />
       </geometry>
     </visual>
@@ -279,5 +279,5 @@
       <origin rpy="0.0 0.0 ${PI}" xyz="0.0 0.0 -${steer_z/2-0.0120}"/>
       <geometry>
-        <mesh filename="package://rm3_sherpa_description/meshes/rbsherpa_hl_steer_wheel.dae" />
+        <mesh filename="package://rm3_sherpa_description/description/meshes/rbsherpa_hl_steer_wheel.dae" />
       </geometry>
     </visual>
@@ -308,5 +308,5 @@
       <origin rpy="0.0 ${PI/2} 0.0" xyz="0.0 -${wheel_width/2} 0.0"/>
       <geometry>
-        <mesh filename="package://rm3_sherpa_description/meshes/rbsherpa_hl_traction_wheel.dae" />
+        <mesh filename="package://rm3_sherpa_description/description/meshes/rbsherpa_hl_traction_wheel.dae" />
       </geometry>
     </visual>
