Commit message: plugin updated

File: description/urdf/arm.xacro (robot description, xacro)
@@ -50,5 +50,5 @@
     <origin xyz="0.0 0.0 ${1.89120-(chassis_z+chassis_field_height)}" rpy="0.0 0.0 0.0"/>
      <axis xyz="0.0 0.0 -1"/>-->
-	<limit effort="100" lower="-3.1415" upper="3.1415" velocity="0.4"/>
+	<limit effort="1000" lower="-3.1415" upper="3.1415" velocity="0.2"/>
 </joint>
 <link name="${prefix}torso_pantilt_pan_link">
