Commit message: moved gazebo camera reference

File: description/urdf/sensors.xacro (robot description, xacro)
@@ -367,6 +367,19 @@
 		<origin xyz="0.11540 0.14610 0.06410" rpy="0.0 0.0 0.0"/>
 	</joint>
-    <!-- camera -->
-    <gazebo reference="camera">
+	<link name="micasense">
+		<visual>
+			<origin xyz="0.0 0.0 0.0" rpy="0.0 0.0 0.0"/>
+			<geometry>
+				<box size="0.020 0.020 0.020"/>
+			</geometry>
+		</visual>
+		<inertial>
+			<mass value="0.5" />
+			<origin xyz="0.0 0.0 0.0" rpy="0.0 0.0 0.0"/>
+			<box_inertia  m="0.5" h="0.020" w ="0.020" d="0.020"/>
+		</inertial>
+	</link>
+    <!-- camera/micasense -->
+    <gazebo reference="micasense">
         <sensor type="camera" name="camera">
           <update_rate>30.0</update_rate>
@@ -397,5 +410,5 @@
             <imageTopicName>image_raw</imageTopicName>
             <cameraInfoTopicName>camera_info</cameraInfoTopicName>
-            <frameName>camera</frameName>
+            <frameName>micasense</frameName>
             <hackBaseline>0.07</hackBaseline>
             <distortionK1>0.0</distortionK1>
@@ -406,18 +419,5 @@
           </plugin>
         </sensor>
-      </gazebo>
-	<link name="micasense">
-		<visual>
-			<origin xyz="0.0 0.0 0.0" rpy="0.0 0.0 0.0"/>
-			<geometry>
-				<box size="0.020 0.020 0.020"/>
-			</geometry>
-		</visual>
-		<inertial>
-			<mass value="0.5" />
-			<origin xyz="0.0 0.0 0.0" rpy="0.0 0.0 0.0"/>
-			<box_inertia  m="0.5" h="0.020" w ="0.020" d="0.020"/>
-		</inertial>
-	</link>
+    </gazebo>
     <!-- IMU -->
 	<joint name="imu_joint" type="fixed">

Commit message: fix slam odom

File: description/urdf/sensors.xacro (robot description, xacro)
@@ -101,5 +101,5 @@
 	    <material>Gazebo/Yellow</material>
 	</gazebo>
-<!-- GPS -->
+<!-- GPS original- ->
 	<joint name="gps_support_joint" type="fixed">
 		<parent link="gps"/>
@@ -127,4 +127,45 @@
 		<child link="gps"/>
 		<origin xyz="0.72090 -0.09320 1.0160" rpy="0 0 0"/>
+	</joint>
+	<link name="gps">
+		<visual>
+			<origin xyz="0 0 0" rpy="0 0 0"/>
+			<geometry>
+        			<cylinder radius="0.090" length="0.040"/>
+			</geometry>
+		</visual>
+		<inertial>
+			<origin xyz="0 0 0" rpy="0 0 0"/>
+			<mass value="0.50" />
+	    		<cylinder_inertia m="0.50" r="0.090" h="0.040"/>
+		</inertial>
+	</link>
+	-->
+	<!-- GPS -->
+	<joint name="gps_support_joint" type="fixed">
+		<parent link="gps"/>
+		<child link="gps_support"/>
+		<origin xyz="0.0 0.0 -0.15" rpy="0 0 0"/>
+	</joint>
+	<link name="gps_support">
+		<visual>
+			<origin xyz="0 0 0" rpy="0 0 0"/>
+			<geometry>
+        			<cylinder radius="0.0090" length="0.30"/>
+			</geometry>
+		</visual>
+		<inertial>
+			<origin xyz="0 0 0" rpy="0 0 0"/>
+			<mass value="0.50" />
+	    		<cylinder_inertia m="0.50" r="0.0090" h="0.30"/>
+		</inertial>
+	</link>
+	<gazebo reference="gps_support">
+        <material>Gazebo/Black</material>
+    </gazebo>
+	<joint name="gps_joint" type="fixed">
+		<parent link="${prefix}base_link"/>
+		<child link="gps"/>
+		<origin xyz="-0.622 0.0 2.150" rpy="0 0 0"/>
 	</joint>
 	<link name="gps">
